File: position_hardware/position_hardware.kicad_sch (KiCad schematic)
At the start: 9 parts, among them J1 Conn_01x12, J8 Conn_01x04, U1 MPU-9250, U9 BMP280

Commit message: add firmware
Parts:
- J1: footprint (none) -> Connector_JST:JST_SH_BM12B-SRSS-TB_1x12-1MP_P1.00mm_Vertical
Changed lines of the file:
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@@
 			)
 		)
-		(property "Footprint" ""
+		(property "Footprint" "Connector_JST:JST_SH_BM12B-SRSS-TB_1x12-1MP_P1.00mm_Vertical"
 			(at 107.95 54.61 0)
 			(effects
